Commit message: adding d435

File: src/hector_models/hector_sensors_description/urdf/realsense_d435_camera.urdf.xacro (robot description, xacro)
@@ -9,110 +9,247 @@
 -->
 <robot xmlns:xacro="http://ros.org/wiki/xacro">
+    <xacro:macro name="gazebo_d435" params="camera_name reference_link topics_ns depth_optical_frame color_optical_frame infrared1_optical_frame infrared2_optical_frame publish_pointcloud:=true" >
+    <!-- Load parameters to model's main link-->
+    <xacro:property name="deg_to_rad" value="0.01745329251994329577" />
+    <gazebo reference="${reference_link}">
+      <self_collide>0</self_collide>
+      <enable_wind>0</enable_wind>
+      <kinematic>0</kinematic>
+      <gravity>1</gravity>
+      <!--<mu>1</mu>-->
+      <mu2>1</mu2>
+      <fdir1>0 0 0</fdir1>
+      <!--<slip1>0</slip1>
+      <slip2>0</slip2>-->
+      <kp>1e+13</kp>
+      <kd>1</kd>
+      <!--<max_vel>0.01</max_vel>
+      <min_depth>0</min_depth>-->
+      <sensor name="${camera_name}color" type="camera">
+        <camera name="${camera_name}">
+          <horizontal_fov>${69.4*deg_to_rad}</horizontal_fov>
+          <image>
+            <width>640</width>
+            <height>480</height>
+            <format>RGB_INT8</format>
+          </image>
+          <clip>
+            <near>0.1</near>
+            <far>100</far>
+          </clip>
+          <noise>
+            <type>gaussian</type>
+            <mean>0.0</mean>
+            <stddev>0.007</stddev>
+          </noise>
+        </camera>
+        <always_on>1</always_on>
+        <update_rate>30</update_rate>
+        <visualize>1</visualize>
+      </sensor>
+      <sensor name="${camera_name}ired1" type="camera">
+        <camera name="${camera_name}">
+          <horizontal_fov>${85.2*deg_to_rad}</horizontal_fov>
+          <image>
+            <width>1280</width>
+            <height>720</height>
+            <format>L_INT8</format>
+          </image>
+          <clip>
+            <near>0.1</near>
+            <far>100</far>
+          </clip>
+          <noise>
+            <type>gaussian</type>
+            <mean>0.0</mean>
+            <stddev>0.05</stddev>
+          </noise>
+        </camera>
+        <always_on>1</always_on>
+        <update_rate>90</update_rate>
+        <visualize>0</visualize>
+      </sensor>
+      <sensor name="${camera_name}ired2" type="camera">
+        <camera name="${camera_name}">
+          <horizontal_fov>${85.2*deg_to_rad}</horizontal_fov>
+          <image>
+            <width>1280</width>
+            <height>720</height>
+            <format>L_INT8</format>
+          </image>
+          <clip>
+            <near>0.1</near>
+            <far>100</far>
+          </clip>
+          <noise>
+            <type>gaussian</type>
+            <mean>0.0</mean>
+            <stddev>0.05</stddev>
+          </noise>
+        </camera>
+        <always_on>1</always_on>
+        <update_rate>90</update_rate>
+        <visualize>0</visualize>
+      </sensor>
+      <sensor name="${camera_name}depth" type="depth">
+        <camera name="${camera_name}">
+          <horizontal_fov>${85.2*deg_to_rad}</horizontal_fov>
+          <image>
+            <width>1280</width>
+            <height>720</height>
+          </image>
+          <clip>
+            <near>0.1</near>
+            <far>100</far>
+          </clip>
+          <noise>
+            <type>gaussian</type>
+            <mean>0.0</mean>
+            <stddev>0.100</stddev>
+          </noise>
+        </camera>
+        <always_on>1</always_on>
+        <update_rate>90</update_rate>
+        <visualize>0</visualize>
+      </sensor>
+    </gazebo>
+    <gazebo>
+      <plugin name="${topics_ns}" filename="librealsense_gazebo_plugin.so">
+        <prefix>${camera_name}</prefix>
+        <depthUpdateRate>30.0</depthUpdateRate>
+        <colorUpdateRate>30.0</colorUpdateRate>
+        <infraredUpdateRate>30.0</infraredUpdateRate>
+        <depthTopicName>depth/image_raw</depthTopicName>
+        <depthCameraInfoTopicName>depth/camera_info</depthCameraInfoTopicName>
+        <colorTopicName>rgb/image_raw</colorTopicName>
+        <colorCameraInfoTopicName>rgb/camera_info</colorCameraInfoTopicName>
+        <infrared1TopicName>infra1/image_raw</infrared1TopicName>
+        <infrared1CameraInfoTopicName>infra1/camera_info</infrared1CameraInfoTopicName>
+        <infrared2TopicName>infra2/image_raw</infrared2TopicName>
+        <infrared2CameraInfoTopicName>infra2/camera_info</infrared2CameraInfoTopicName>
+        <colorOpticalframeName>${color_optical_frame}</colorOpticalframeName>
+        <depthOpticalframeName>${depth_optical_frame}</depthOpticalframeName>
+        <infrared1OpticalframeName>${infrared1_optical_frame}</infrared1OpticalframeName>
+        <infrared2OpticalframeName>${infrared2_optical_frame}</infrared2OpticalframeName>
+        <rangeMinDepth>0.2</rangeMinDepth>
+        <rangeMaxDepth>10.0</rangeMaxDepth>
+        <pointCloud>${publish_pointcloud}</pointCloud>
+        <pointCloudTopicName>/depth/points</pointCloudTopicName>
+        <pointCloudCutoff>0.25</pointCloudCutoff>
+        <pointCloudCutoffMax>9.0</pointCloudCutoffMax>
+      </plugin>
+    </gazebo>
+  </xacro:macro>
+  <xacro:macro name="sensor_d435" params="name:=camera topics_ns:=camera parent *origin publish_pointcloud:=true">
     <xacro:property name="M_PI" value="3.1415926535897931" />
-    <!--
-     This macro only adds the model, it does not also add
-     the openni gazebo plugin. See the 'asus_camera' macro below for that
-    -->
-    <xacro:macro name="realsense_d435_camera_model" params="name parent *origin">
-      <joint name="${name}_joint" type="fixed">
-        <xacro:insert_block name="origin" />
-        <parent link="${parent}"/>
-        <child link="${name}_link"/>
-      </joint>
-      <link name="${name}_link">
-        <inertial>
-          <mass value="0.072" />
-          <origin xyz="0 0 0" rpy="0 0 0" />
-          <inertia ixx="5.8083e-4" ixy="0" ixz="0" iyy="3.0833e-5" iyz="0" izz="5.9083e-4" />
-        </inertial>
-        <visual>
-          <origin xyz="0 0.0115 0" rpy="0 0 0" />
-          <geometry>
-            <!--Dimensions taken from https://click.intel.com/intelr-realsensetm-depth-camera-d435.html-->
-            <box size="0.025 0.09 0.025" />
-          </geometry>
-          <material name="DarkGrey">
-            <color rgba="0.3 0.3 0.3 1"/>
-          </material>
-        </visual>
-        <collision>
-          <origin xyz="0 0.0115 0" rpy="0 0 0" />
-          <geometry>
-            <!--Dimensions taken from https://click.intel.com/intelr-realsensetm-depth-camera-d435.html-->
-            <box size="0.025 0.09 0.025" />
-          </geometry>update_rate
-        </collision>
-      </link>
-      <gazebo reference="${name}_link">
-        <material>Gazebo/Grey</material>
-      </gazebo>
-    </xacro:macro>
-    <xacro:macro name="realsense_d435_camera_model_no_geom" params="name parent *origin">
-      <joint name="${name}_joint" type="fixed">
-        <xacro:insert_block name="origin" />
-        <parent link="${parent}"/>
-        <child link="${name}_link"/>
-      </joint>
-      <link name="${name}_link">
-      </link>
-    </xacro:macro>
-    <xacro:macro name="realsense_d435_camera_gazebo_plugin_macro" params="name parent image_topic depth_points_topic min_range max_range update_rate">
-      <gazebo reference="${name}_link">
-        <sensor type="depth" name="${name}">
-          <update_rate>${update_rate}</update_rate>
-          <camera>
-            <horizontal_fov>${69.4 * M_PI/180.0}</horizontal_fov>
-            <image>
-              <format>B8G8R8</format>
-              <width>848</width>
-              <height>480</height>
-            </image>
-            <clip>
-              <near>${min_range}</near>
-              <far>${max_range}</far>
-            </clip>
-          </camera>
-          <plugin name="${name}_camera_controller" filename="libgazebo_ros_openni_kinect.so">
-            <cameraName>${name}</cameraName>
-            <imageTopicName>rgb/${image_topic}</imageTopicName>
-            <cameraInfoTopicName>rgb/camera_info</cameraInfoTopicName>
-            <depthImageTopicName>depth/image_raw</depthImageTopicName>
-            <depthImageCameraInfoTopicName>depth/camera_info</depthImageCameraInfoTopicName>
-            <pointCloudTopicName>${depth_points_topic}</pointCloudTopicName>
-            <frameName>${name}_depth_optical_frame</frameName>
-          </plugin>
-        </sensor>
-      </gazebo>
-    </xacro:macro>
-    <!--
-      Use the macro below for adding the realsense model with link geometry
-    -->
-    <xacro:macro name="realsense_d435_camera" params="name parent *origin">
-      <xacro:realsense_d435_camera_model name="${name}" parent="${parent}">
-        <xacro:insert_block name="origin" />
-      </xacro:realsense_d435_camera_model>
-      <xacro:realsense_d435_camera_gazebo_plugin_macro name="${name}" parent="${parent}" image_topic="rgb/image_raw" depth_points_topic="depth/points" min_range="0.3" max_range="9.0" update_rate="20"/>
-    </xacro:macro>
-    <!--
-      Use the macro below for adding the realsense model without link geometry,
-      e.g. if the sensor is added into preexisting geometry
-    -->
-    <xacro:macro name="realsense_camera_no_geom" params="name parent *origin">
-      <xacro:realsense_d435_camera_model_no_geom name="${name}" parent="${parent}">
-        <xacro:insert_block name="origin" />
-      </xacro:realsense_d435_camera_model_no_geom>
-      <xacro:realsense_camera_gazebo_plugin_macro name="${name}" parent="${parent}" image_topic="rgb/image_raw" depth_points_topic="depth/points" min_range="0.3" max_range="9.0" update_rate="20"/>
-    </xacro:macro>
-    <xacro:macro name="realsense_d435_camera_no_geom_comprehensive_params" params="name parent *origin image_topic depth_points_topic min_range max_range update_rate">
-      <xacro:realsense_d435_camera_model_no_geom name="${name}" parent="${parent}">
-        <xacro:insert_block name="origin" />
-      </xacro:realsense_d435_camera_model_no_geom>
-      <xacro:realsense_camera_gazebo_plugin_macro name="${name}" parent="${parent}" image_topic="${image_topic}" depth_points_topic="${depth_points_topic}" min_range="${min_range}" max_range="${max_range}" update_rate="${update_rate}"/>
-    </xacro:macro>
-    <xacro:macro name="realsense_d435_camera_comprehensive_params" params="name parent *origin image_topic depth_points_topic min_range max_range update_rate">
-      <xacro:realsense_d435_camera_model name="${name}" parent="${parent}">
-        <xacro:insert_block name="origin" />
-      </xacro:realsense_d435_camera_model>
-      <xacro:realsense_d435_camera_gazebo_plugin_macro name="${name}" parent="${parent}" image_topic="${image_topic}" depth_points_topic="${depth_points_topic}" min_range="${min_range}" max_range="${max_range}" update_rate="${update_rate}"/>
-    </xacro:macro>
+    <!-- The following values are approximate, and the camera node
+     publishing TF values with actual calibrated camera extrinsic values -->
+    <xacro:property name="d435_cam_depth_to_left_ir_offset" value="0.0"/>
+    <xacro:property name="d435_cam_depth_to_right_ir_offset" value="-0.050"/>
+    <xacro:property name="d435_cam_depth_to_color_offset" value="0.015"/>
+    <!-- The following values model the aluminum peripherial case for the
+    D435 camera, with the camera joint represented by the actual
+    peripherial camera tripod mount -->
+    <xacro:property name="d435_cam_width" value="0.090"/>
+    <xacro:property name="d435_cam_height" value="0.025"/>
+    <xacro:property name="d435_cam_depth" value="0.02505"/>
+    <xacro:property name="d435_cam_mount_from_center_offset" value="0.0149"/>
+    <!-- The following offset is relative the the physical D435 camera peripherial
+    camera tripod mount -->
+    <xacro:property name="d435_cam_depth_px" value="${d435_cam_mount_from_center_offset}"/>
+    <xacro:property name="d435_cam_depth_py" value="0.0175"/>
+    <xacro:property name="d435_cam_depth_pz" value="${d435_cam_height/2}"/>
+    <material name="${name}_aluminum">
+    <color rgba="0.5 0.5 0.5 1"/>
+    </material>
+    <!-- camera body, with origin at bottom screw mount -->
+    <joint name="${name}_joint" type="fixed">
+      <xacro:insert_block name="origin" />
+      <parent link="${parent}"/>
+      <child link="${name}_bottom_screw_frame" />
+    </joint>
+    <link name="${name}_bottom_screw_frame"/>
+    <joint name="${name}_link_joint" type="fixed">
+      <origin xyz="0 ${d435_cam_depth_py} ${d435_cam_depth_pz}" rpy="0 0 0"/>
+      <parent link="${name}_bottom_screw_frame"/>
+      <child link="${name}_link" />
+    </joint>
+    <link name="${name}_link">
+      <visual>
+      <origin xyz="${d435_cam_mount_from_center_offset} ${-d435_cam_depth_py} 0" rpy="${M_PI/2} 0 ${M_PI/2}"/>
+        <geometry>
+          <!-- <box size="${d435_cam_width} ${d435_cam_height} ${d435_cam_depth}"/> -->
+          <mesh filename="package://realsense2_description/meshes/d435.dae" />
+          <!--<mesh filename="package://realsense2_description/meshes/d435/d435.dae" />-->
+        </geometry>
+        <material name="${name}_aluminum"/>
+      </visual>
+      <collision>
+        <origin xyz="0 ${-d435_cam_depth_py} 0" rpy="0 0 0"/>
+        <geometry>
+        <box size="${d435_cam_depth} ${d435_cam_width} ${d435_cam_height}"/>
+        </geometry>
+      </collision>
+      <inertial>
+        <!-- The following are not reliable values, and should not be used for modeling -->
+        <mass value="0.564" />
+        <origin xyz="0 0 0" />
+        <inertia ixx="0.003881243" ixy="0.0" ixz="0.0" iyy="0.000498940" iyz="0.0" izz="0.003879257" />
+      </inertial>
+    </link>
+    <!-- camera depth joints and links -->
+    <joint name="${name}_depth_joint" type="fixed">
+      <origin xyz="0 0 0" rpy="0 0 0"/>
+      <parent link="${name}_link"/>
+      <child link="${name}_depth_frame" />
+    </joint>
+    <link name="${name}_depth_frame"/>
+    <joint name="${name}_depth_optical_joint" type="fixed">
+      <origin xyz="0 0 0" rpy="${-M_PI/2} 0 ${-M_PI/2}" />
+      <parent link="${name}_depth_frame" />
+      <child link="${name}_depth_optical_frame" />
+    </joint>
+    <link name="${name}_depth_optical_frame"/>
+    <!-- camera left IR joints and links -->
+    <joint name="${name}_left_ir_joint" type="fixed">
+      <origin xyz="0 ${d435_cam_depth_to_left_ir_offset} 0" rpy="0 0 0" />
+      <parent link="${name}_depth_frame" />
+      <child link="${name}_left_ir_frame" />
+    </joint>
+    <link name="${name}_left_ir_frame"/>
+    <joint name="${name}_left_ir_optical_joint" type="fixed">
+      <origin xyz="0 0 0" rpy="${-M_PI/2} 0 ${-M_PI/2}" />
+      <parent link="${name}_left_ir_frame" />
+      <child link="${name}_left_ir_optical_frame" />
+    </joint>
+    <link name="${name}_left_ir_optical_frame"/>
+    <!-- camera right IR joints and links -->
+    <joint name="${name}_right_ir_joint" type="fixed">
+      <origin xyz="0 ${d435_cam_depth_to_right_ir_offset} 0" rpy="0 0 0" />
+      <parent link="${name}_depth_frame" />
+      <child link="${name}_right_ir_frame" />
+    </joint>
+    <link name="${name}_right_ir_frame"/>
+    <joint name="${name}_right_ir_optical_joint" type="fixed">
+      <origin xyz="0 0 0" rpy="${-M_PI/2} 0 ${-M_PI/2}" />
+      <parent link="${name}_right_ir_frame" />
+      <child link="${name}_right_ir_optical_frame" />
+    </joint>
+    <link name="${name}_right_ir_optical_frame"/>
+    <!-- camera color joints and links -->
+    <joint name="${name}_color_joint" type="fixed">
+      <origin xyz="0 ${d435_cam_depth_to_color_offset} 0" rpy="0 0 0" />
+      <parent link="${name}_depth_frame" />
+      <child link="${name}_color_frame" />
+    </joint>
+    <link name="${name}_color_frame"/>
+    <joint name="${name}_color_optical_joint" type="fixed">
+      <origin xyz="0 0 0" rpy="${-M_PI/2} 0 ${-M_PI/2}" />
+      <parent link="${name}_color_frame" />
+      <child link="${name}_color_optical_frame" />
+    </joint>
+    <link name="${name}_color_optical_frame"/>
+    <!-- Realsense Gazebo Plugin -->
+    <xacro:gazebo_d435 camera_name="${name}" reference_link="${name}_link" topics_ns="${topics_ns}" depth_optical_frame="${name}_depth_optical_frame" color_optical_frame="${name}_color_optical_frame" infrared1_optical_frame="${name}_left_ir_optical_frame" infrared2_optical_frame="${name}_right_ir_optical_frame" publish_pointcloud="${publish_pointcloud}"/>
+  </xacro:macro>
   </robot>

File: src/hector_quadrotor/hector_quadrotor_description/urdf/quadrotor_with_kinect.urdf.xacro (robot description, xacro)
@@ -7,7 +7,7 @@
     <xacro:quadrotor_base_macro />
     <!-- Kinect -->
-    <xacro:include filename="$(find hector_sensors_description)/urdf/kinect_camera.urdf.xacro" />
-    <xacro:kinect_camera name="camera" parent="base_link">
+    <xacro:include filename="$(find hector_sensors_description)/urdf/realsense_d435_camera.urdf.xacro" />
+    <xacro:sensor_d435 name="camera" parent="base_link">
       <origin xyz="0.23 0.0 -0.1" rpy="0 0 0"/>
-    </xacro:kinect_camera>
+    </xacro:sensor_d435>
 </robot>

Commit message: Editing the mass of the camera

File: src/hector_models/hector_sensors_description/urdf/realsense_d435_camera.urdf.xacro (robot description, xacro)
@@ -193,5 +193,5 @@
       <inertial>
         <!-- The following are not reliable values, and should not be used for modeling -->
-        <mass value="0.564" />
+        <mass value="0.12" />
         <origin xyz="0 0 0" />
         <inertia ixx="0.003881243" ixy="0.0" ixz="0.0" iyy="0.000498940" iyz="0.0" izz="0.003879257" />
